Commit message: now featuring slam

File: description/robot_core.xacro (robot description, xacro)
@@ -21,4 +21,12 @@
     <!--the rest of the robot will be described w.r. to base_link-->
     <link name="base_link">
+    </link>
+    <!-- BASE_FOOTPRINT LINK -->
+    <joint name="base_footprint_joint" type="fixed">
+        <parent link="base_link"/>
+        <child link="base_footprint"/>
+        <origin xyz="0 0 0" rpy="0 0 0"/>
+    </joint>
+    <link name="base_footprint">
     </link>
     <!-- CHASSIS LINK -->
