Commit message: update robot geometry

File: description/lidar.xacro (robot description, xacro)
@@ -4,5 +4,5 @@
         <parent link="chassis"/>
         <child link="laser_frame"/>
-        <origin xyz="0.1 0 0.1625" rpy="0 0 0"/>
+        <origin xyz="0.1016 0 0.1625" rpy="0 0 0"/>
     </joint>
     <link name="laser_frame">
@@ -26,5 +26,5 @@
         <sensor name="laser" type="ray">
             <pose> 0 0 0 0 0 0 </pose>
-            <visualize>true</visualize>
+            <visualize>false</visualize>
             <update_rate>10</update_rate>
             <ray>

File: description/robot.urdf.xacro (robot description, xacro)
@@ -11,3 +11,4 @@
     </xacro:unless>
     <xacro:include filename="lidar.xacro" />
+    <xacro:include filename="camera.xacro"/> <!--safe to use but camera functionality incomplete-->
 </robot>

File: description/robot_core.xacro (robot description, xacro)
@@ -2,4 +2,18 @@
 <robot xmlns:xacro="http://www.ros.org/wiki/xacro" >
     <xacro:include filename="inertial_macros.xacro"/>
+    <xacro:property name="chassis_length" value="0.2032"/>
+    <xacro:property name="chassis_width" value="0.1524"/>
+    <xacro:property name="chassis_height" value="0.1397"/>
+    <xacro:property name="chassis_mass" value="1.0"/>
+    <xacro:property name="wheel_radius" value="0.04445"/>
+    <xacro:property name="wheel_thickness" value="0.01215"/>
+    <xacro:property name="wheel_mass" value="0.01"/>
+    <xacro:property name="wheel_offset_x" value="0.0635"/>
+    <xacro:property name="wheel_offset_y" value="0.1143"/>
+    <xacro:property name="wheel_offset_z" value="0.0381"/>
+    <xacro:property name="caster_wheel_radius" value="0.014"/>
+    <xacro:property name="caster_wheel_mass" value="0.01"/>
+    <xacro:property name="caster_wheel_offset_x" value="0.1715"/>
+    <xacro:property name="caster_wheel_offset_z" value="${wheel_offset_z - wheel_radius + caster_wheel_radius}"/>
     <material name="white">
         <color rgba="1 1 1 1" />
@@ -35,5 +49,5 @@
         <child link="chassis"/>
         <!--need to adjust origin to align wheels on chassis-->
-        <origin xyz="-0.04 0 0"/>
+        <origin xyz="${-wheel_offset_x} 0 ${-wheel_offset_z}"/>
     </joint>
     <link name="chassis">
@@ -41,18 +55,18 @@
             <!--need to adjust origin of chassis box to align robopet wheel positions-->
             <!--need to change box geometry, collision, and inertial tags-->
-            <origin xyz="0.115 0 0.075"/>
+            <origin xyz="${chassis_length/2} 0 ${chassis_height/2}"/>
             <geometry>
-                <box size="0.23 0.15 0.15"/>
+                <box size="${chassis_length} ${chassis_width} ${chassis_height}"/>
             </geometry>
             <material name="white"/>
         </visual>
         <collision>
-            <origin xyz="0.115 0 0.075"/>
+            <origin xyz="${chassis_length/2} 0 ${chassis_height/2}"/>
             <geometry>
-                <box size="0.23 0.15 0.15"/>
+                <box size="${chassis_length} ${chassis_width} ${chassis_height}"/>
             </geometry>
         </collision>
-        <xacro:inertial_box mass="0.5" x="0.23" y="0.15" z="0.15">
-            <origin xyz="0.115 0 0.075" rpy="0 0 0"/>
+        <xacro:inertial_box mass="0.5" x="${chassis_length}" y="${chassis_width}" z="${chassis_height}">
+            <origin xyz="${chassis_length/2} 0 ${chassis_height/2}" rpy="0 0 0"/>
         </xacro:inertial_box>
     </link>
@@ -65,5 +79,5 @@
         <child link="left_wheel"/>
         <!--adjust wheel joint origin to proper chassis width-->
-        <origin xyz="0 0.1 0" rpy="-${pi/2} 0 0"/>
+        <origin xyz="0 ${wheel_offset_y} 0" rpy="-${pi/2} 0 0"/>
         <axis xyz="0 0 1"/>
     </joint>
@@ -72,5 +86,5 @@
         <visual>
             <geometry>
-                <cylinder radius="0.03" length="0.025"/>
+                <cylinder radius="${wheel_radius}" length="${wheel_thickness}"/>
             </geometry>
             <material name="blue"/>
@@ -78,8 +92,8 @@
         <collision>
             <geometry>
-                <sphere radius="0.03"/>
+                <sphere radius="${wheel_radius}"/>
             </geometry>
         </collision>
-        <xacro:inertial_cylinder mass="0.1" length="0.025" radius="0.03">
+        <xacro:inertial_cylinder mass="${wheel_mass}" length="${wheel_thickness}" radius="${wheel_radius}">
             <origin xyz="0 0 0" rpy="0 0 0"/>
         </xacro:inertial_cylinder>
@@ -93,5 +107,5 @@
         <child link="right_wheel"/>
         <!--adjust wheel joint origin to proper chassis width-->
-        <origin xyz="0 -0.1 0" rpy="${pi/2} 0 0"/>
+        <origin xyz="0 ${-wheel_offset_y} 0" rpy="${pi/2} 0 0"/>
         <axis xyz="0 0 -1"/>
     </joint>
@@ -100,5 +114,5 @@
         <visual>
             <geometry>
-                <cylinder radius="0.03" length="0.025"/>
+                <cylinder radius="${wheel_radius}" length="${wheel_thickness}"/>
             </geometry>
             <material name="blue"/>
@@ -106,8 +120,8 @@
         <collision>
             <geometry>
-                <sphere radius="0.03"/>
+                <sphere radius="${wheel_radius}"/>
             </geometry>
         </collision>
-        <xacro:inertial_cylinder mass="0.1" length="0.025" radius="0.03">
+        <xacro:inertial_cylinder mass="${wheel_mass}" length="${wheel_thickness}" radius="${wheel_radius}">
             <origin xyz="0 0 0" rpy="0 0 0"/>
         </xacro:inertial_cylinder>
@@ -122,5 +136,5 @@
         <child link="caster_wheel"/>
         <!--may adjust origin to align it on bot-->
-        <origin xyz="0.2 0 0"/>
+        <origin xyz="${caster_wheel_offset_x} 0 ${caster_wheel_offset_z}"/>
     </joint>
     <link name="caster_wheel">
@@ -128,5 +142,5 @@
         <visual>
             <geometry>
-                <sphere radius="0.03"/>
+                <sphere radius="${caster_wheel_radius}"/>
             </geometry>
             <material name="black"/>
@@ -134,8 +148,8 @@
         <collision>
             <geometry>
-                <sphere radius="0.03"/>
+                <sphere radius="${caster_wheel_radius}"/>
             </geometry>
         </collision>
-        <xacro:inertial_sphere mass="0.1" radius="0.03">
+        <xacro:inertial_sphere mass="${caster_wheel_mass}" radius="${caster_wheel_radius}">
             <origin xyz="0 0 0" rpy="0 0 0"/>
         </xacro:inertial_sphere>

File: description/ros2_control.xacro (robot description, xacro)
@@ -8,5 +8,5 @@
                 <param name="right_wheel_name">right_wheel_joint</param>
                 <param name="loop_rate">30</param>
-                <param name="device">/dev/ttyUSB0</param>   <!--may need to change to prevent conflicts with rplidar-->
+                <param name="device">/dev/ttyUSB0</param>   <!--arduino is ttyUSB0 and lidar is ttyUSB1-->
                 <param name="baud_rate">57600</param>
                 <param name="timeout">1000</param>
